File: Eagle/GaragentorSteuerung.brd (EAGLE design)
At the start: 100.3 x 80 mm, 11 parts

Commit message: V0.1
sync
Parts:
- moved JP2 2.84 mm to (30.5, 3.81)
- moved OK3 2.54 mm to (30.5, 25.4)
- moved OK1 2.54 mm to (38.1, 17.8)
- moved OK4 2.54 mm to (22.9, 25.4)
- moved R1 2.54 mm to (39.4, 34.3)
- moved R3 2.54 mm to (29.2, 12.7)
Connections:
- removed net N$10: R1.1, U$1.D0
- new net N$15: JP2.3, U$1.D7
- new net N$16: S2.2
- net N$1: now also U$1.D8; no longer U$1.D2
- net N$4: now also OK4.4, U$1.D6; no longer JP2.3, U$1.D1
- net N$8: now also OK3.4, U$1.D5; no longer OK4.4, U$1.D4
- net N$9: now also R1.1, U$1.D1; no longer OK3.4, U$1.D3
Routing:
- net N$15: track 0.00 -> 41.3 mm
- net N$4: track 43.6 -> 12.9 mm
- net N$9: track 13.7 -> 4.04 mm
- net N$1: track 44.6 -> 40.3 mm
- net N$10: track 4.00 -> 0.00 mm
- net N$2: track 46.7 -> 48.9 mm
- net N$7: track 31.2 -> 33.1 mm
- net N$11: track 11.7 -> 10.2 mm
- net N$5: track 30.2 -> 28.8 mm
- net N$13: track 6.35 -> 5.10 mm
- net N$12: track 11.6 -> 10.4 mm
- net N$8: track 15.9 -> 14.9 mm
