File: Eagle/GaragentorSteuerung.sch (EAGLE design)
At the start: 11 parts

Commit message: V0.1
sync
Connections:
- removed net N$10: R1.1, U$1.D0
- new net N$15: JP2.3, U$1.D7
- new net N$16: S2.S1
- net N$1: now also U$1.D8; no longer U$1.D2
- net N$4: now also OK4.COL, U$1.D6; no longer JP2.3, U$1.D1
- net N$8: now also OK3.COL, U$1.D5; no longer OK4.COL, U$1.D4
- net N$9: now also R1.1, U$1.D1; no longer OK3.COL, U$1.D3
Other:
- moved on the sheet: JP2, OK3, OK4, R3
